Commit message: fixed color

File: description/model_generic/model_generic_aCol.urdf (robot description, URDF)
Before this commit: robot model_generic, 23 links, 22 joints
Joints:
- joint ground_pelvis: origin xyz= 0.00000000  0.00000000  0.00000000 rpy=0 0 0 -> xyz= 1.00000000  1.00000000  1.00000000 rpy=0 0 0

Commit message: changed package name

File: description/model_generic/model_generic_aCol.urdf (robot description, URDF)
Before this commit: robot model_generic, 23 links, 22 joints
Links:
- link calcn_l: geometry collision box size=0.0849 0.1936 0.0529; visual mesh filename=package://gait1992_description/description/model_generic/st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 scale=1.00000000 1.00000000 1.00000000
- link calcn_r: geometry collision box size=0.0849 0.1927 0.0529; visual mesh filename=package://gait1992_description/description/model_generic/st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 scale=1.00000000 1.00000000 1.00000000
- link femur_l: geometry collision cylinder length=0.452616 radius=0.043163001537323; visual mesh filename=package://gait1992_description/description/model_generic/st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 scale=1.00000000 1.00000000 1.00000000
- link femur_r: geometry collision cylinder length=0.452616 radius=0.043163001537323; visual mesh filename=package://gait1992_description/description/model_generic/st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 scale=1.00000000 1.00000000 1.00000000
- link pelvis: geometry collision cylinder length=0.21470201 radius=0.06901049613952637; collision cylinder length=0.21470201 radius=0.06901049613952637
- link talus_l: geometry collision box size=0.0416 0.0461 0.0301; visual mesh filename=package://gait1992_description/description/model_generic/st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 scale=1.00000000 1.00000000 1.00000000
- link talus_r: geometry collision box size=0.0416 0.0458 0.0301; visual mesh filename=package://gait1992_description/description/model_generic/st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 scale=1.00000000 1.00000000 1.00000000
- link tibia_l: geometry collision cylinder length=0.375208 radius=0.014540750533342361; collision cylinder length=0.386749 radius=0.034585751593112946
- link tibia_r: geometry collision cylinder length=0.375208 radius=0.014540750533342361; collision cylinder length=0.386749 radius=0.034585751593112946
- link toes_l: geometry collision cylinder length=0.018185 radius=0.05118675157427788; visual mesh filename=package://gait1992_description/description/model_generic/st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 scale=1.00000000 1.00000000 1.00000000
- link toes_r: geometry collision cylinder length=0.018185 radius=0.05094899982213974; visual mesh filename=package://gait1992_description/description/model_generic/st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 scale=1.00000000 1.00000000 1.00000000
- link torso: geometry collision box size=0.0751 0.1291 0.5249; collision box size=0.2758 0.1928 0.3097
