Commit message: attempt at fixing tfs

File: description/model_generic/model_generic.urdf.xacro (robot description, xacro)
@@ -8,4 +8,5 @@
 		</gazebo>
 		<link name="${parent}" />
+		<link name="urdf_pelvis" />
 		<link name="pelvis">
 			<inertial>
@@ -377,7 +378,12 @@
 			</collision>
 		</link>
-		<joint name="ground_pelvis" type="floating">
-			<origin xyz=" 1.00000000  1.00000000  1.00000000" rpy="0 0 0" />
-			<parent link="ground"/>
+		<joint name="pelvis_urdf_joint" type="floating">
+			<origin xyz=" 0 0 0 " rpy="0 0 0" />
+			<parent link="${parent}"/>
+			<child link="urdf_pelvis"/>
+		</joint>
+		<joint name="rotate_pelvis" type="fixed">
+			<origin xyz="0 0 0" rpy="-1.57079633 -1.57079633 0" />
+			<parent link="urdf_pelvis"/>
 			<child link="pelvis"/>
 		</joint>

Commit message: removed unused frame urdf_pelvis

File: description/model_generic/model_generic.urdf.xacro (robot description, xacro)
@@ -8,5 +8,4 @@
 		</gazebo>
 		<link name="${parent}" />
-		<link name="urdf_pelvis" />
 		<link name="pelvis">
 			<inertial>
@@ -378,12 +377,7 @@
 			</collision>
 		</link>
-		<joint name="pelvis_urdf_joint" type="floating">
-			<origin xyz=" 0 0 0 " rpy="0 0 0" />
-			<parent link="${parent}"/>
-			<child link="urdf_pelvis"/>
-		</joint>
 		<joint name="rotate_pelvis" type="fixed">
 			<origin xyz="0 0 0" rpy="-1.57079633 -1.57079633 0" />
-			<parent link="urdf_pelvis"/>
+			<parent link="${parent}"/>
 			<child link="pelvis"/>
 		</joint>

Commit message: Does this make it better?

File: description/model_generic/model_generic.urdf.xacro (robot description, xacro)
@@ -377,5 +377,5 @@
 			</collision>
 		</link>
-		<joint name="rotate_pelvis" type="fixed">
+		<joint name="rotate_pelvis" type="floating">
 			<origin xyz="0 0 0" rpy="-1.57079633 -1.57079633 0" />
 			<parent link="${parent}"/>

Commit message: did something, now they are revolute, but the fixed tf publishers will likely complain or be unnecessary

File: description/model_generic/model_generic.urdf.xacro (robot description, xacro)
@@ -529,13 +529,17 @@
 			</actuator>
 		</transmission>
-		<joint name="subtalar_r" type="floating">
+		<joint name="subtalar_r" type="revolute">
 			<origin xyz=" 0.00792000 -0.04877000 -0.04195000" rpy="0 0 0" />
 			<parent link="talus_r"/>
 			<child link="calcn_r"/>
-		</joint>
-		<joint name="mtp_r" type="floating">
+			<axis xyz="0.0 1.0 0.0"/>
+			<limit effort="23.648" velocity="1.0" lower="-1.57079633" upper="1.57079633" />
+		</joint>
+		<joint name="mtp_r" type="revolute">
 			<origin xyz=" 0.00108000  0.17880000 -0.00200000" rpy="0 0 0" />
 			<parent link="calcn_r"/>
 			<child link="toes_r"/>
+			<axis xyz="1.0 0.0 0.0"/>
+			<limit effort="23.648" velocity="1.0" lower="-1.57079633" upper="1.57079633" />
 		</joint>
 		<link name="femur_l_f1">
@@ -686,13 +690,17 @@
 			</actuator>
 		</transmission>
-		<joint name="subtalar_l" type="floating">
+		<joint name="subtalar_l" type="revolute">
 			<origin xyz="-0.00792000 -0.04877000 -0.04195000" rpy="0 0 0" />
 			<parent link="talus_l"/>
 			<child link="calcn_l"/>
-		</joint>
-		<joint name="mtp_l" type="floating">
+			<axis xyz="0.0 1.0 0.0"/>
+			<limit effort="23.648" velocity="1.0" lower="-1.57079633" upper="1.57079633" />
+		</joint>
+		<joint name="mtp_l" type="revolute">
 			<origin xyz="-0.00108000  0.17880000 -0.00200000" rpy="0 0 0" />
 			<parent link="calcn_l"/>
 			<child link="toes_l"/>
+			<axis xyz="1.0 0.0 0.0"/>
+			<limit effort="23.648" velocity="1.0" lower="-1.57079633" upper="1.57079633" />
 		</joint>
 		<link name="torso_f1">
