Commit message: shows almost ok, still need to fix subject_opensim frame and IMU orientations

File: description/model_generic/model_generic.urdf.xacro (robot description, xacro)
@@ -1,5 +1,5 @@
 <?xml version="1.0" ?>
 <robot name="model_generic" xmlns:xacro="http://www.ros.org/wiki/xacro">
-	<xacro:macro name="a_human" params="parent">
+	<xacro:macro name="a_human" params="parent color:=1 global_scale:=0.92">
 		<gazebo>
 			<plugin name="gazebo_ros_control" filename="libgazebo_ros_control.so">
@@ -11,18 +11,18 @@
 			<inertial>
 				<mass value="11.777"/>
-				<origin xyz="-0.00000000 -0.07070000  0.00000000" rpy="0 0 0" />
+				<origin xyz="${-0.00000000*global_scale} ${-0.07070000*global_scale} ${0.00000000*global_scale}" rpy="0 0 0" />
 				<inertia ixx="0.1028" iyy="0.0871" izz="0.0579" ixy="0.0" ixz="0.0" iyz="0.0"/>
 			</inertial>
 			<visual name="sacrum">
-				<origin xyz=" 0.00000000  0.00000000  0.00000000" rpy=" 1.57079633 -0.00000000  1.57079633" />
-				<geometry>
-					<mesh filename="package://gait1992_description/description/model_generic/stl/sacrum.stl" scale=" 1.00000000  1.00000000  1.00000000"/>
-				</geometry>
-				<material name="">
-					<color rgba="0.792156862745098 0.819607843137255 0.933333333333333 1" />
+				<origin xyz="${0.00000000*global_scale} ${0.00000000*global_scale} ${0.00000000*global_scale}" rpy=" 1.57079633 -0.00000000  1.57079633" />
+				<geometry>
+					<mesh filename="package://gait1992_description/description/model_generic/stl/sacrum.stl" scale = "${global_scale} ${global_scale} ${global_scale}"/>
+				</geometry>
+				<material name="">
+					<color rgba="${0.792156862745098*color} 0.819607843137255 0.933333333333333 1" />
 				</material>
 			</visual>
 			<collision name="sacrum">
-				<origin xyz=" 0.00000889 -0.12485057  0.03677944" rpy=" 0.00000000  0.00000000  0.00000000" />
+				<origin xyz="${0.00000889*global_scale} ${-0.12485057*global_scale} ${0.03677944*global_scale}" rpy=" 0.00000000  0.00000000  0.00000000" />
 				<geometry>
 					<sphere radius="0.0528053343296051" />
@@ -30,14 +30,14 @@
 			</collision>
 			<visual name="pelvis">
-				<origin xyz=" 0.00000000  0.00000000  0.00000000" rpy=" 1.57079633 -0.00000000  1.57079633" />
-				<geometry>
-					<mesh filename="package://gait1992_description/description/model_generic/stl/pelvis.stl" scale=" 1.00000000  1.00000000  1.00000000"/>
-				</geometry>
-				<material name="">
-					<color rgba="0.792156862745098 0.819607843137255 0.933333333333333 1" />
+				<origin xyz="${0.00000000*global_scale} ${0.00000000*global_scale} ${0.00000000*global_scale}" rpy=" 1.57079633 -0.00000000  1.57079633" />
+				<geometry>
+					<mesh filename="package://gait1992_description/description/model_generic/stl/pelvis.stl" scale = "${global_scale} ${global_scale} ${global_scale}"/>
+				</geometry>
+				<material name="">
+					<color rgba="${0.792156862745098*color} 0.819607843137255 0.933333333333333 1" />
 				</material>
 			</visual>
 			<collision name="pelvis">
-				<origin xyz=" 0.07386850 -0.07562926 -0.00743482" rpy=" 0.00000000  0.00000000  0.00000000" />
+				<origin xyz="${0.07386850*global_scale} ${-0.07562926*global_scale} ${-0.00743482*global_scale}" rpy=" 0.00000000  0.00000000  0.00000000" />
 				<geometry>
 					<cylinder radius="0.06901049613952637" length="0.21470201" />
@@ -45,14 +45,14 @@
 			</collision>
 			<visual name="l_pelvis">
-				<origin xyz=" 0.00000000  0.00000000  0.00000000" rpy=" 1.57079633 -0.00000000  1.57079633" />
-				<geometry>
-					<mesh filename="package://gait1992_description/description/model_generic/stl/l_pelvis.stl" scale=" 1.00000000  1.00000000  1.00000000"/>
-				</geometry>
-				<material name="">
-					<color rgba="0.792156862745098 0.819607843137255 0.933333333333333 1" />
+				<origin xyz="${0.00000000*global_scale} ${0.00000000*global_scale} ${0.00000000*global_scale}" rpy=" 1.57079633 -0.00000000  1.57079633" />
+				<geometry>
+					<mesh filename="package://gait1992_description/description/model_generic/stl/l_pelvis.stl" scale = "${global_scale} ${global_scale} ${global_scale}"/>
+				</geometry>
+				<material name="">
+					<color rgba="${0.792156862745098*color} 0.819607843137255 0.933333333333333 1" />
 				</material>
 			</visual>
 			<collision name="l_pelvis">
-				<origin xyz="-0.07386850 -0.07562925 -0.00743482" rpy=" 0.00000000  0.00000000  0.00000000" />
+				<origin xyz="${-0.07386850*global_scale} ${-0.07562925*global_scale} ${-0.00743482*global_scale}" rpy=" 0.00000000  0.00000000  0.00000000" />
 				<geometry>
 					<cylinder radius="0.06901049613952637" length="0.21470201" />
@@ -63,18 +63,18 @@
 			<inertial>
 				<mass value="9.3014"/>
-				<origin xyz=" 0.00000000 -0.00000000 -0.17000000" rpy="0 0 0" />
+				<origin xyz="${0.00000000*global_scale} ${-0.00000000*global_scale} ${-0.17000000*global_scale}" rpy="0 0 0" />
 				<inertia ixx="0.1339" iyy="0.0351" izz="0.1412" ixy="0.0" ixz="0.0" iyz="0.0"/>
 			</inertial>
 			<visual name="femur_r">
-				<origin xyz=" 0.00000000  0.00000000  0.00000000" rpy=" 1.57079633 -0.00000000  1.57079633" />
-				<geometry>
-					<mesh filename="package://gait1992_description/description/model_generic/stl/femur_r.stl" scale=" 1.00000000  1.00000000  1.00000000"/>
-				</geometry>
-				<material name="">
-					<color rgba="0.792156862745098 0.819607843137255 0.933333333333333 1" />
+				<origin xyz="${0.00000000*global_scale} ${0.00000000*global_scale} ${0.00000000*global_scale}" rpy=" 1.57079633 -0.00000000  1.57079633" />
+				<geometry>
+					<mesh filename="package://gait1992_description/description/model_generic/stl/femur_r.stl" scale = "${global_scale} ${global_scale} ${global_scale}"/>
+				</geometry>
+				<material name="">
+					<color rgba="${0.792156862745098*color} 0.819607843137255 0.933333333333333 1" />
 				</material>
 			</visual>
 			<collision name="femur_r">
-				<origin xyz=" 0.01594298  0.00497468 -0.20699716" rpy=" 0.00000000  0.00000000  0.00000000" />
+				<origin xyz="${0.01594298*global_scale} ${0.00497468*global_scale} ${-0.20699716*global_scale}" rpy=" 0.00000000  0.00000000  0.00000000" />
 				<geometry>
 					<cylinder radius="0.043163001537323" length="0.452616" />
@@ -85,18 +85,18 @@
 			<inertial>
 				<mass value="3.7075"/>
-				<origin xyz=" 0.00000000 -0.00000000 -0.18670000" rpy="0 0 0" />
+				<origin xyz="${0.00000000*global_scale} ${-0.00000000*global_scale} ${-0.18670000*global_scale}" rpy="0 0 0" />
 				<inertia ixx="0.0504" iyy="0.0051" izz="0.0511" ixy="0.0" ixz="0.0" iyz="0.0"/>
 			</inertial>
 			<visual name="tibia_r">
-				<origin xyz=" 0.00000000  0.00000000  0.00000000" rpy=" 1.57079633 -0.00000000  1.57079633" />
-				<geometry>
-					<mesh filename="package://gait1992_description/description/model_generic/stl/tibia_r.stl" scale=" 1.00000000  1.00000000  1.00000000"/>
-				</geometry>
-				<material name="">
-					<color rgba="0.792156862745098 0.819607843137255 0.933333333333333 1" />
+				<origin xyz="${0.00000000*global_scale} ${0.00000000*global_scale} ${0.00000000*global_scale}" rpy=" 1.57079633 -0.00000000  1.57079633" />
+				<geometry>
+					<mesh filename="package://gait1992_description/description/model_generic/stl/tibia_r.stl" scale = "${global_scale} ${global_scale} ${global_scale}"/>
+				</geometry>
+				<material name="">
+					<color rgba="${0.792156862745098*color} 0.819607843137255 0.933333333333333 1" />
 				</material>
 			</visual>
 			<collision name="tibia_r">
-				<origin xyz="-0.00346711  0.00744511 -0.18540447" rpy=" 0.00000000  0.00000000  0.00000000" />
+				<origin xyz="${-0.00346711*global_scale} ${0.00744511*global_scale} ${-0.18540447*global_scale}" rpy=" 0.00000000  0.00000000  0.00000000" />
 				<geometry>
 					<cylinder radius="0.034585751593112946" length="0.386749" />
@@ -104,14 +104,14 @@
 			</collision>
 			<visual name="fibula">
-				<origin xyz=" 0.00000000  0.00000000  0.00000000" rpy=" 1.57079633 -0.00000000  1.57079633" />
-				<geometry>
-					<mesh filename="package://gait1992_description/description/model_generic/stl/fibula.stl" scale=" 1.00000000  1.00000000  1.00000000"/>
-				</geometry>
-				<material name="">
-					<color rgba="0.792156862745098 0.819607843137255 0.933333333333333 1" />
+				<origin xyz="${0.00000000*global_scale} ${0.00000000*global_scale} ${0.00000000*global_scale}" rpy=" 1.57079633 -0.00000000  1.57079633" />
+				<geometry>
+					<mesh filename="package://gait1992_description/description/model_generic/stl/fibula.stl" scale = "${global_scale} ${global_scale} ${global_scale}"/>
+				</geometry>
+				<material name="">
+					<color rgba="${0.792156862745098*color} 0.819607843137255 0.933333333333333 1" />
 				</material>
 			</visual>
 			<collision name="fibula">
-				<origin xyz=" 0.03035371 -0.00401039 -0.23035097" rpy=" 0.00000000  0.00000000  0.00000000" />
+				<origin xyz="${0.03035371*global_scale} ${-0.00401039*global_scale} ${-0.23035097*global_scale}" rpy=" 0.00000000  0.00000000  0.00000000" />
 				<geometry>
 					<cylinder radius="0.014540750533342361" length="0.375208" />
@@ -122,18 +122,19 @@
 			<inertial>
 				<mass value="0.1"/>
-				<origin xyz=" 0.00000000  0.00000000  0.00000000" rpy="0 0 0" />
+				<origin xyz="${0.00000000*global_scale} ${0.00000000*global_scale} ${0.00000000*global_scale}" rpy="0 0 0" />
 				<inertia ixx="0.001" iyy="0.001" izz="0.001" ixy="0.0" ixz="0.0" iyz="0.0"/>
 			</inertial>
 			<visual name="talus">
-				<origin xyz=" 0.00000000  0.00000000  0.00000000" rpy=" 1.57079633 -0.00000000  1.57079633" />
-				<geometry>
-					<mesh filename="package://gait1992_description/description/model_generic/stl/talus.stl" scale=" 1.00000000  1.00000000  1.00000000"/>
-				</geometry>
-				<material name="">
-					<color rgba="0.792156862745098 0.819607843137255 0.933333333333333 1" />
+				<origin xyz="${0.00000000*global_scale} ${0.00000000*global_scale} ${0.00000000*global_scale}" rpy=" 1.57079633 -0.00000000  1.57079633" />
+				<geometry>
+					<mesh filename="package://gait1992_description/description/model_generic/stl/talus.stl" scale = "${global_scale} ${global_scale} ${global_scale}"/>
+				</geometry>
+				<material name="">
+					<color rgba="${0.792156862745098*color} 0.819607843137255 0.933333333333333 1" />
 				</material>
 			</visual>
 			<collision name="talus">
-				<origin xyz="-0.00168721  0.00594951  0.00035094" rpy=" 0.00000000  0.00000000  0.00000000" />
+				2j
+				<origin xyz="${-0.00168721*global_scale} ${0.00594951*global_scale} ${0.00035094*global_scale}" rpy=" 0.00000000  0.00000000  0.00000000" />
 				<geometry>
 					<box size=" 0.0416  0.0458  0.0301" />
@@ -144,18 +145,18 @@
 			<inertial>
 				<mass value="1.25"/>
-				<origin xyz=" 0.00000000  0.10000000  0.03000000" rpy="0 0 0" />
+				<origin xyz="${0.00000000*global_scale} ${0.10000000*global_scale} ${0.03000000*global_scale}" rpy="0 0 0" />
 				<inertia ixx="0.0014" iyy="0.0039" izz="0.0041" ixy="0.0" ixz="0.0" iyz="0.0"/>
 			</inertial>
 			<visual name="foot">
-				<origin xyz=" 0.00000000  0.00000000  0.00000000" rpy=" 1.57079633 -0.00000000  1.57079633" />
-				<geometry>
-					<mesh filename="package://gait1992_description/description/model_generic/stl/foot.stl" scale=" 1.00000000  1.00000000  1.00000000"/>
-				</geometry>
-				<material name="">
-					<color rgba="0.792156862745098 0.819607843137255 0.933333333333333 1" />
+				<origin xyz="${0.00000000*global_scale} ${0.00000000*global_scale} ${0.00000000*global_scale}" rpy=" 1.57079633 -0.00000000  1.57079633" />
+				<geometry>
+					<mesh filename="package://gait1992_description/description/model_generic/stl/foot.stl" scale = "${global_scale} ${global_scale} ${global_scale}"/>
+				</geometry>
+				<material name="">
+					<color rgba="${0.792156862745098*color} 0.819607843137255 0.933333333333333 1" />
 				</material>
 			</visual>
 			<collision name="foot">
-				<origin xyz="-0.00432009  0.07068449  0.01758767" rpy=" 0.00000000  0.00000000  0.00000000" />
+				<origin xyz="${-0.00432009*global_scale} ${0.07068449*global_scale} ${0.01758767*global_scale}" rpy=" 0.00000000  0.00000000  0.00000000" />
 				<geometry>
 					<box size=" 0.0849  0.1927  0.0529" />
@@ -166,18 +167,18 @@
 			<inertial>
 				<mass value="0.2166"/>
-				<origin xyz="-0.01750000  0.03460000  0.00600000" rpy="0 0 0" />
+				<origin xyz="${-0.01750000*global_scale} ${0.03460000*global_scale} ${0.00600000*global_scale}" rpy="0 0 0" />
 				<inertia ixx="0.0001" iyy="0.0002" izz="0.0001" ixy="0.0" ixz="0.0" iyz="0.0"/>
 			</inertial>
 			<visual name="bofoot">
-				<origin xyz=" 0.00000000  0.00000000  0.00000000" rpy=" 1.57079633 -0.00000000  1.57079633" />
-				<geometry>
-					<mesh filename="package://gait1992_description/description/model_generic/stl/bofoot.stl" scale=" 1.00000000  1.00000000  1.00000000"/>
-				</geometry>
-				<material name="">
-					<color rgba="0.792156862745098 0.819607843137255 0.933333333333333 1" />
+				<origin xyz="${0.00000000*global_scale} ${0.00000000*global_scale} ${0.00000000*global_scale}" rpy=" 1.57079633 -0.00000000  1.57079633" />
+				<geometry>
+					<mesh filename="package://gait1992_description/description/model_generic/stl/bofoot.stl" scale = "${global_scale} ${global_scale} ${global_scale}"/>
+				</geometry>
+				<material name="">
+					<color rgba="${0.792156862745098*color} 0.819607843137255 0.933333333333333 1" />
 				</material>
 			</visual>
 			<collision name="bofoot">
-				<origin xyz="-0.00004618  0.02500000 -0.00304539" rpy=" 0.00000000  0.00000000  0.00000000" />
+				<origin xyz="${-0.00004618*global_scale} ${0.02500000*global_scale} ${-0.00304539*global_scale}" rpy=" 0.00000000  0.00000000  0.00000000" />
 				<geometry>
 					<cylinder radius="0.05094899982213974" length="0.018185" />
@@ -188,18 +189,18 @@
 			<inertial>
 				<mass value="9.3014"/>
-				<origin xyz=" 0.00000000 -0.00000000 -0.17000000" rpy="0 0 0" />
+				<origin xyz="${0.00000000*global_scale} ${-0.00000000*global_scale} ${-0.17000000*global_scale}" rpy="0 0 0" />
 				<inertia ixx="0.1339" iyy="0.0351" izz="0.1412" ixy="0.0" ixz="0.0" iyz="0.0"/>
 			</inertial>
 			<visual name="femur_l">
-				<origin xyz=" 0.00000000  0.00000000  0.00000000" rpy=" 1.57079633 -0.00000000  1.57079633" />
-				<geometry>
-					<mesh filename="package://gait1992_description/description/model_generic/stl/femur_l.stl" scale=" 1.00000000  1.00000000  1.00000000"/>
-				</geometry>
-				<material name="">
-					<color rgba="0.792156862745098 0.819607843137255 0.933333333333333 1" />
+				<origin xyz="${0.00000000*global_scale} ${0.00000000*global_scale} ${0.00000000*global_scale}" rpy=" 1.57079633 -0.00000000  1.57079633" />
+				<geometry>
+					<mesh filename="package://gait1992_description/description/model_generic/stl/femur_l.stl" scale = "${global_scale} ${global_scale} ${global_scale}"/>
+				</geometry>
+				<material name="">
+					<color rgba="${0.792156862745098*color} 0.819607843137255 0.933333333333333 1" />
 				</material>
 			</visual>
 			<collision name="femur_l">
-				<origin xyz="-0.01594298  0.00497468 -0.20699715" rpy=" 0.00000000  0.00000000  0.00000000" />
+				<origin xyz="${-0.01594298*global_scale} ${0.00497468*global_scale} ${-0.20699715*global_scale}" rpy=" 0.00000000  0.00000000  0.00000000" />
 				<geometry>
 					<cylinder radius="0.043163001537323" length="0.452616" />
@@ -210,18 +211,18 @@
 			<inertial>
 				<mass value="3.7075"/>
-				<origin xyz=" 0.00000000 -0.00000000 -0.18670000" rpy="0 0 0" />
+				<origin xyz="${0.00000000*global_scale} ${-0.00000000*global_scale} ${-0.18670000*global_scale}" rpy="0 0 0" />
 				<inertia ixx="0.0504" iyy="0.0051" izz="0.0511" ixy="0.0" ixz="0.0" iyz="0.0"/>
 			</inertial>
 			<visual name="tibia_l">
-				<origin xyz=" 0.00000000  0.00000000  0.00000000" rpy=" 1.57079633 -0.00000000  1.57079633" />
-				<geometry>
-					<mesh filename="package://gait1992_description/description/model_generic/stl/tibia_l.stl" scale=" 1.00000000  1.00000000  1.00000000"/>
-				</geometry>
-				<material name="">
-					<color rgba="0.792156862745098 0.819607843137255 0.933333333333333 1" />
+				<origin xyz="${0.00000000*global_scale} ${0.00000000*global_scale} ${0.00000000*global_scale}" rpy=" 1.57079633 -0.00000000  1.57079633" />
+				<geometry>
+					<mesh filename="package://gait1992_description/description/model_generic/stl/tibia_l.stl" scale = "${global_scale} ${global_scale} ${global_scale}"/>
+				</geometry>
+				<material name="">
+					<color rgba="${0.792156862745098*color} 0.819607843137255 0.933333333333333 1" />
 				</material>
 			</visual>
 			<collision name="tibia_l">
-				<origin xyz=" 0.00346711  0.00744511 -0.18540446" rpy=" 0.00000000  0.00000000  0.00000000" />
+				<origin xyz="${0.00346711*global_scale} ${0.00744511*global_scale} ${-0.18540446*global_scale}" rpy=" 0.00000000  0.00000000  0.00000000" />
 				<geometry>
 					<cylinder radius="0.034585751593112946" length="0.386749" />
@@ -229,14 +230,14 @@
 			</collision>
 			<visual name="l_fibula">
-				<origin xyz=" 0.00000000  0.00000000  0.00000000" rpy=" 1.57079633 -0.00000000  1.57079633" />
-				<geometry>
-					<mesh filename="package://gait1992_description/description/model_generic/stl/l_fibula.stl" scale=" 1.00000000  1.00000000  1.00000000"/>
-				</geometry>
-				<material name="">
-					<color rgba="0.792156862745098 0.819607843137255 0.933333333333333 1" />
+				<origin xyz="${0.00000000*global_scale} ${0.00000000*global_scale} ${0.00000000*global_scale}" rpy=" 1.57079633 -0.00000000  1.57079633" />
+				<geometry>
+					<mesh filename="package://gait1992_description/description/model_generic/stl/l_fibula.stl" scale = "${global_scale} ${global_scale} ${global_scale}"/>
+				</geometry>
+				<material name="">
+					<color rgba="${0.792156862745098*color} 0.819607843137255 0.933333333333333 1" />
 				</material>
 			</visual>
 			<collision name="l_fibula">
-				<origin xyz="-0.03035371 -0.00401039 -0.23035097" rpy=" 0.00000000  0.00000000  0.00000000" />
+				<origin xyz="${-0.03035371*global_scale} ${-0.00401039*global_scale} ${-0.23035097*global_scale}" rpy=" 0.00000000  0.00000000  0.00000000" />
 				<geometry>
 					<cylinder radius="0.014540750533342361" length="0.375208" />
@@ -247,18 +248,18 @@
 			<inertial>
 				<mass value="0.1"/>
-				<origin xyz=" 0.00000000  0.00000000  0.00000000" rpy="0 0 0" />
+				<origin xyz="${0.00000000*global_scale} ${0.00000000*global_scale} ${0.00000000*global_scale}" rpy="0 0 0" />
 				<inertia ixx="0.001" iyy="0.001" izz="0.001" ixy="0.0" ixz="0.0" iyz="0.0"/>
 			</inertial>
 			<visual name="l_talus">
-				<origin xyz=" 0.00000000  0.00000000  0.00000000" rpy=" 1.57079633 -0.00000000  1.57079633" />
-				<geometry>
-					<mesh filename="package://gait1992_description/description/model_generic/stl/l_talus.stl" scale=" 1.00000000  1.00000000  1.00000000"/>
-				</geometry>
-				<material name="">
-					<color rgba="0.792156862745098 0.819607843137255 0.933333333333333 1" />
+				<origin xyz="${0.00000000*global_scale} ${0.00000000*global_scale} ${0.00000000*global_scale}" rpy=" 1.57079633 -0.00000000  1.57079633" />
+				<geometry>
+					<mesh filename="package://gait1992_description/description/model_generic/stl/l_talus.stl" scale = "${global_scale} ${global_scale} ${global_scale}"/>
+				</geometry>
+				<material name="">
+					<color rgba="${0.792156862745098*color} 0.819607843137255 0.933333333333333 1" />
 				</material>
 			</visual>
 			<collision name="l_talus">
-				<origin xyz=" 0.00168721  0.00594951  0.00035094" rpy=" 0.00000000  0.00000000  0.00000000" />
+				<origin xyz="${0.00168721*global_scale} ${0.00594951*global_scale} ${0.00035094*global_scale}" rpy=" 0.00000000  0.00000000  0.00000000" />
 				<geometry>
 					<box size=" 0.0416  0.0461  0.0301" />
@@ -269,18 +270,18 @@
 			<inertial>
 				<mass value="1.25"/>
-				<origin xyz=" 0.00000000  0.10000000  0.03000000" rpy="0 0 0" />
+				<origin xyz="${0.00000000*global_scale} ${0.10000000*global_scale} ${0.03000000*global_scale}" rpy="0 0 0" />
 				<inertia ixx="0.0014" iyy="0.0039" izz="0.0041" ixy="0.0" ixz="0.0" iyz="0.0"/>
 			</inertial>
 			<visual name="l_foot">
-				<origin xyz=" 0.00000000  0.00000000  0.00000000" rpy=" 1.57079633 -0.00000000  1.57079633" />
-				<geometry>
-					<mesh filename="package://gait1992_description/description/model_generic/stl/l_foot.stl" scale=" 1.00000000  1.00000000  1.00000000"/>
-				</geometry>
-				<material name="">
-					<color rgba="0.792156862745098 0.819607843137255 0.933333333333333 1" />
+				<origin xyz="${0.00000000*global_scale} ${0.00000000*global_scale} ${0.00000000*global_scale}" rpy=" 1.57079633 -0.00000000  1.57079633" />
+				<geometry>
+					<mesh filename="package://gait1992_description/description/model_generic/stl/l_foot.stl" scale = "${global_scale} ${global_scale} ${global_scale}"/>
+				</geometry>
+				<material name="">
+					<color rgba="${0.792156862745098*color} 0.819607843137255 0.933333333333333 1" />
 				</material>
 			</visual>
 			<collision name="l_foot">
-				<origin xyz=" 0.00432009  0.07068449  0.01758767" rpy=" 0.00000000  0.00000000  0.00000000" />
+				<origin xyz="${0.00432009*global_scale} ${0.07068449*global_scale} ${0.01758767*global_scale}" rpy=" 0.00000000  0.00000000  0.00000000" />
 				<geometry>
 					<box size=" 0.0849  0.1936  0.0529" />
@@ -291,18 +292,18 @@
 			<inertial>
 				<mass value="0.2166"/>
-				<origin xyz=" 0.01750000  0.03460000  0.00600000" rpy="0 0 0" />
+				<origin xyz="${0.01750000*global_scale} ${0.03460000*global_scale} ${0.00600000*global_scale}" rpy="0 0 0" />
 				<inertia ixx="0.0001" iyy="0.0002" izz="0.0001" ixy="0.0" ixz="0.0" iyz="0.0"/>
 			</inertial>
 			<visual name="l_bofoot">
-				<origin xyz=" 0.00000000  0.00000000  0.00000000" rpy=" 1.57079633 -0.00000000  1.57079633" />
-				<geometry>
-					<mesh filename="package://gait1992_description/description/model_generic/stl/l_bofoot.stl" scale=" 1.00000000  1.00000000  1.00000000"/>
-				</geometry>
-				<material name="">
-					<color rgba="0.792156862745098 0.819607843137255 0.933333333333333 1" />
+				<origin xyz="${0.00000000*global_scale} ${0.00000000*global_scale} ${0.00000000*global_scale}" rpy=" 1.57079633 -0.00000000  1.57079633" />
+				<geometry>
+					<mesh filename="package://gait1992_description/description/model_generic/stl/l_bofoot.stl" scale = "${global_scale} ${global_scale} ${global_scale}"/>
+				</geometry>
+				<material name="">
+					<color rgba="${0.792156862745098*color} 0.819607843137255 0.933333333333333 1" />
 				</material>
 			</visual>
 			<collision name="l_bofoot">
-				<origin xyz="-0.00073217  0.02228543 -0.00115883" rpy=" 0.00000000  0.00000000  0.00000000" />
+				<origin xyz="${-0.00073217*global_scale} ${0.02228543*global_scale} ${-0.00115883*global_scale}" rpy=" 0.00000000  0.00000000  0.00000000" />
 				<geometry>
 					<cylinder radius="0.05118675157427788" length="0.018185" />
@@ -313,18 +314,18 @@
 			<inertial>
 				<mass value="34.2366"/>
-				<origin xyz="-0.00000000 -0.03000000  0.32000000" rpy="0 0 0" />
+				<origin xyz="${-0.00000000*global_scale} ${-0.03000000*global_scale} ${0.32000000*global_scale}" rpy="0 0 0" />
 				<inertia ixx="1.4745" iyy="0.7555" izz="1.4314" ixy="0.0" ixz="0.0" iyz="0.0"/>
 			</inertial>
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