Commit message: removed redundant? joint and link

File: description/model_generic/model_generic.urdf.xacro (robot description, xacro)
@@ -7,5 +7,4 @@
 			</plugin>
 		</gazebo>
-		<link name="${parent}" />
 		<link name="pelvis">
 			<inertial>
@@ -378,9 +377,4 @@
 			</collision>
 		</link>
-		<joint name="rotate_pelvis" type="floating">
-			<origin xyz="${0*global_scale} ${0*global_scale} ${0*global_scale}" rpy="-1.57079633 -1.57079633 0" />
-			<parent link="${parent}"/>
-			<child link="pelvis"/>
-		</joint>
 		<link name="femur_r_f1">
 			<inertial>
