Commit message: removed some hardcoded paths

File: description/model_generic/human_with_ximus_movable.urdf.xacro (robot description, xacro)
@@ -2,5 +2,5 @@
 <robot xmlns:xacro="http://ros.org/wiki/xacro" name="model_generic">
 	<xacro:include filename="$(find gait1992_description)/description/model_generic/model_generic.urdf.xacro" />
-	<xacro:a_human parent="subject_opensim" />
+	<xacro:a_human parent="subject_opensim" global_scale="$(arg scale)"/>
 	<xacro:include filename="$(find ximu3_ros)/urdf/ximu3.urdf.xacro" />
 	<xacro:ximu_link_and_joint_floating parent="torso" origin="0 -0.1 0.3" />

File: description/model_generic/model_generic.urdf.xacro (robot description, xacro)
@@ -1,5 +1,5 @@
 <?xml version="1.0" ?>
 <robot name="model_generic" xmlns:xacro="http://www.ros.org/wiki/xacro">
-	<xacro:macro name="a_human" params="parent color:=1 global_scale:=0.92">
+	<xacro:macro name="a_human" params="parent color:=1 global_scale:=^|0.921">
 		<gazebo>
 			<plugin name="gazebo_ros_control" filename="libgazebo_ros_control.so">
